File: hardware/industrial-ptc.kicad_pcb (KiCad board)
At the start: 2 copper layers, 40 x 40 mm, 35 parts, among them P1 CON-SENSOR, P2 Debug, P3 Boot, P4 CONN_01X08, SW1 SW_DIP_4, SW2 SW_DIP_4, U1 XMC1100, U2 MAX31865, U3 DRILL, U4 DRILL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

Commit message: ready for prototype
Other:
- board text added: "Industrial PTC 1.0"
- board text removed: "Ind. PTC 2.0"
Changed lines of the file:
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@@
     (title "Industrial PTC Bricklet")
     (date 2020-06-18)
-    (rev 2.0)
+    (rev 1.0)
     (company "Tinkerforge GmbH")
     (comment 1 "Licensed under CERN OHL v.1.1")
@@
     (31 Rückseite signal)
     (32 B.Adhes user)
-    (33 F.Adhes user hide)
+    (33 F.Adhes user)
     (34 B.Paste user)
     (35 F.Paste user)
@@
     (43 Eco2.User user)
     (44 Edge.Cuts user)
+    (45 Margin user)
+    (46 B.CrtYd user)
+    (47 F.CrtYd user)
     (48 B.Fab user)
     (49 F.Fab user)
   )
   (setup
-    (last_trace_width 0.15)
+    (last_trace_width 0.29972)
     (user_trace_width 0.15)
     (user_trace_width 0.29972)
@@
     (pad_drill 0)
     (pad_to_mask_clearance 0)
-    (solder_mask_min_width 0.25)
     (aux_axis_origin 124.9 69.95)
     (grid_origin 124.9 69.95)
@@
     (effects (font (size 0.8001 0.8001) (thickness 0.14986)))
   )
-  (gr_text Status (at 163.9 81.05 270) (layer F.SilkS)
+  (gr_text Status (at 161.6 78.25 270) (layer F.SilkS)
     (effects (font (size 0.8001 0.8001) (thickness 0.14986)))
   )
@@
     (effects (font (size 1.04902 1.04902) (thickness 0.2)))
   )
-  (gr_text "Ind. PTC 2.0" (at 163.9 100.85 270) (layer F.SilkS)
+  (gr_text "Industrial\n PTC 1.0" (at 162.3 100.75 270) (layer F.SilkS)
     (effects (font (size 0.8001 0.8001) (thickness 0.14986)))
   )
-  (gr_text "Sensor\nType" (at 148.99924 107.70044 270) (layer F.SilkS)
+  (gr_text "Sensor\nType" (at 148.99924 107.45 270) (layer F.SilkS)
     (effects (font (size 0.8001 0.8001) (thickness 0.14986)))
   )
@@
   (segment (start 142.67 89.82) (end 141.3 88.45) (width 0.8001) (layer Rückseite) (net 2))
   (segment (start 142.67 97.14) (end 142.67 89.82) (width 0.8001) (layer Rückseite) (net 2))
+  (segment (start 132.94982 95.25) (end 132.9 95.20018) (width 0.8001) (layer Vorderseite) (net 3))
+  (segment (start 140.2889 91.5474) (end 139.6 92.2363) (width 0.29972) (layer Vorderseite) (net 3))
+  (segment (start 139.6 92.2363) (end 139.6 92.55) (width 0.29972) (layer Vorderseite) (net 3))
+  (segment (start 141.16266 91.5474) (end 140.2889 91.5474) (width 0.29972) (layer Vorderseite) (net 3))
+  (segment (start 135.7 102.87) (end 135.7 95.20018) (width 0.8001) (layer Rückseite) (net 3))
+  (segment (start 137.59 104.76) (end 135.7 102.87) (width 0.8001) (layer Rückseite) (net 3))
+  (segment (start 132.9 95.20018) (end 135.7 95.20018) (width 0.8001) (layer Vorderseite) (net 3))
+  (via (at 135.7 95.20018) (size 0.7) (drill 0.25) (layers Vorderseite Rückseite) (net 3))
+  (segment (start 136.194974 95.20018) (end 135.7 95.20018) (width 0.8001) (layer Vorderseite) (net 3))
+  (segment (start 136.94982 95.20018) (end 136.194974 95.20018) (width 0.8001) (layer Vorderseite) (net 3))
+  (segment (start 139.79315 92.04315) (end 139.79315 92.35685) (width 0.8001) (layer Vorderseite) (net 3))
+  (segment (start 139.79315 92.35685) (end 136.94982 95.20018) (width 0.8001) (layer Vorderseite) (net 3))
+  (segment (start 145.21 104.76) (end 142.67 104.76) (width 0.8001) (layer Rückseite) (net 4))
+  (via (at 139.6 89.05) (size 0.7) (drill 0.25) (layers Vorderseite Rückseite) (net 4))
+  (segment (start 139.6 89.05) (end 140.1 89.05) (width 0.59944) (layer Vorderseite) (net 4))
+  (segment (start 140.1 89.05) (end 140.5 89.45) (width 0.59944) (layer Vorderseite) (net 4))
+  (segment (start 140.65176 89.60176) (end 140.5 89.45) (width 0.29972) (layer Vorderseite) (net 4))
+  (segment (start 141.16266 89.60176) (end 140.65176 89.60176) (width 0.29972) (layer Vorderseite) (net 4))
+  (segment (start 141.4 90.85) (end 139.6 89.05) (width 0.59944) (layer Rückseite) (net 4))
+  (segment (start 141.4 103.49) (end 141.4 90.85) (width 0.59944) (layer Rückseite) (net 4))
+  (segment (start 142.67 104.76) (end 141.4 103.49) (width 0.59944) (layer Rückseite) (net 4))
   (segment (start 157.95 79.275) (end 157.95 78.35) (width 0.29972) (layer Vorderseite) (net 5))
   (segment (start 157.95 78.35) (end 158.2 78.1) (width 0.29972) (layer Vorderseite) (net 5))
@@
   (via (at 163.7 94.8) (size 0.7) (drill 0.25) (layers Vorderseite Rückseite) (net 5))
   (segment (start 163.69902 94.80098) (end 163.7 94.8) (width 0.59944) (layer Vorderseite) (net 5))
-  (segment (start 132.94982 95.25) (end 132.9 95.20018) (width 0.8001) (layer Vorderseite) (net 3))
-  (segment (start 140.2889 91.5474) (end 139.6 92.2363) (width 0.29972) (layer Vorderseite) (net 3))
-  (segment (start 139.6 92.2363) (end 139.6 92.55) (width 0.29972) (layer Vorderseite) (net 3))
-  (segment (start 141.16266 91.5474) (end 140.2889 91.5474) (width 0.29972) (layer Vorderseite) (net 3))
-  (segment (start 135.7 102.87) (end 135.7 95.20018) (width 0.8001) (layer Rückseite) (net 3))
-  (segment (start 137.59 104.76) (end 135.7 102.87) (width 0.8001) (layer Rückseite) (net 3))
-  (segment (start 132.9 95.20018) (end 135.7 95.20018) (width 0.8001) (layer Vorderseite) (net 3))
-  (via (at 135.7 95.20018) (size 0.7) (drill 0.25) (layers Vorderseite Rückseite) (net 3))
-  (segment (start 136.194974 95.20018) (end 135.7 95.20018) (width 0.8001) (layer Vorderseite) (net 3))
-  (segment (start 136.94982 95.20018) (end 136.194974 95.20018) (width 0.8001) (layer Vorderseite) (net 3))
-  (segment (start 139.79315 92.04315) (end 139.79315 92.35685) (width 0.8001) (layer Vorderseite) (net 3))
-  (segment (start 139.79315 92.35685) (end 136.94982 95.20018) (width 0.8001) (layer Vorderseite) (net 3))
-  (segment (start 145.21 104.76) (end 142.67 104.76) (width 0.8001) (layer Rückseite) (net 4))
-  (via (at 139.6 89.05) (size 0.7) (drill 0.25) (layers Vorderseite Rückseite) (net 4))
-  (segment (start 139.6 89.05) (end 140.1 89.05) (width 0.59944) (layer Vorderseite) (net 4))
-  (segment (start 140.1 89.05) (end 140.5 89.45) (width 0.59944) (layer Vorderseite) (net 4))
-  (segment (start 140.65176 89.60176) (end 140.5 89.45) (width 0.29972) (layer Vorderseite) (net 4))
-  (segment (start 141.16266 89.60176) (end 140.65176 89.60176) (width 0.29972) (layer Vorderseite) (net 4))
-  (segment (start 141.4 90.85) (end 139.6 89.05) (width 0.59944) (layer Rückseite) (net 4))
-  (segment (start 141.4 103.49) (end 141.4 90.85) (width 0.59944) (layer Rückseite) (net 4))
-  (segment (start 142.67 104.76) (end 141.4 103.49) (width 0.59944) (layer Rückseite) (net 4))
   (via (at 151.3 84.25) (size 0.7) (drill 0.25) (layers Vorderseite Rückseite) (net 5))
   (segment (start 150.45 84.25) (end 151.3 84.25) (width 0.8001) (layer Vorderseite) (net 5))
